File: ToolHead/LowPowerPWM.kicad_sch (KiCad schematic)
At the start: 7 parts, among them J5 Conn_01x02, Q4 ES3400

Commit message: Moderate update. Moving to other computer.
Parts:
- renumbered D9 to D5, D10 to D6, Q4 to Q2, R16 to R10, R17 to R11, R18 to R12
Changed lines of the file:
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@@
   (symbol (lib_id "Device:R_Small") (at 30.226 41.656 90) (unit 1)
     (in_bom yes) (on_board yes) (fields_autoplaced)
-    (property "Reference" "R16" (id 0) (at 30.226 36.322 90))
+    (property "Reference" "R10" (id 0) (at 30.226 36.322 90))
     (property "Value" "22" (id 1) (at 30.226 38.862 90))
     (property "Footprint" "Resistor_SMD:R_0603_1608Metric_Pad0.98x0.95mm_HandSolder" (id 2) (at 30.226 41.656 0)
@@
   (symbol (lib_id "Device:R_Small") (at 30.226 50.038 90) (unit 1)
     (in_bom yes) (on_board yes) (fields_autoplaced)
-    (property "Reference" "R17" (id 0) (at 30.226 44.704 90))
+    (property "Reference" "R11" (id 0) (at 30.226 44.704 90))
     (property "Value" "10k" (id 1) (at 30.226 47.244 90))
     (property "Footprint" "Resistor_SMD:R_0603_1608Metric_Pad0.98x0.95mm_HandSolder" (id 2) (at 30.226 50.038 0)
@@
   (symbol (lib_id "Device:R_Small") (at 39.624 23.622 0) (unit 1)
     (in_bom yes) (on_board yes) (fields_autoplaced)
-    (property "Reference" "R18" (id 0) (at 41.91 22.3519 0)
+    (property "Reference" "R12" (id 0) (at 41.91 22.3519 0)
       (effects (font (size 1.27 1.27)) (justify left))
     )
@@
   (symbol (lib_id "Device:D_Small") (at 47.244 27.432 270) (unit 1)
     (in_bom yes) (on_board yes) (fields_autoplaced)
-    (property "Reference" "D10" (id 0) (at 49.276 26.1619 90)
+    (property "Reference" "D6" (id 0) (at 49.276 26.1619 90)
       (effects (font (size 1.27 1.27)) (justify left))
     )
@@
   (symbol (lib_id "Device:LED_Small") (at 39.624 30.988 90) (unit 1)
     (in_bom yes) (on_board yes) (fields_autoplaced)
-    (property "Reference" "D9" (id 0) (at 41.656 29.6544 90)
+    (property "Reference" "D5" (id 0) (at 41.656 29.6544 90)
       (effects (font (size 1.27 1.27)) (justify right))
     )
@@
   (symbol (lib_id "Device:Q_NMOS_DGS") (at 40.894 41.656 0) (unit 1)
     (in_bom yes) (on_board yes) (fields_autoplaced)
-    (property "Reference" "Q4" (id 0) (at 46.736 40.3859 0)
+    (property "Reference" "Q2" (id 0) (at 46.736 40.3859 0)
       (effects (font (size 1.27 1.27)) (justify left))
     )
@@
   (symbol (lib_id "power:GND") (at 43.434 51.562 0) (unit 1)
     (in_bom yes) (on_board yes) (fields_autoplaced)
-    (property "Reference" "#PWR0112" (id 0) (at 43.434 57.912 0)
+    (property "Reference" "#PWR0110" (id 0) (at 43.434 57.912 0)
       (effects (font (size 1.27 1.27)) hide)
     )
