File: ToolHead/ToolHead.kicad_pcb (KiCad board)
At the start: 2 copper layers, 44 parts, among them J1 CANBUS, J2 Conn_01x02_Male, J3 Conn_01x02_Male, J4 Conn_01x02, J5 Conn_01x02, J6 Conn_01x02, J7 Conn_01x02, J8 Conn_01x02, J9 Conn_01x04, U1 ADXL345

Commit message: Moderate update. Moving to other computer.
Parts:
- added C10: C_Small, Capacitor_SMD:C_0603_1608Metric_Pad1.08x0.95mm_HandSolder, F.Cu at (26.8, 21.2)
- added C3: C_Small, Capacitor_SMD:C_0603_1608Metric_Pad1.08x0.95mm_HandSolder, F.Cu at (25.6, 30.6)
- added C4: C_Small, Capacitor_SMD:C_0603_1608Metric_Pad1.08x0.95mm_HandSolder, F.Cu at (16.8, 31.8)
- added C5: C_Small, Capacitor_SMD:C_0603_1608Metric_Pad1.08x0.95mm_HandSolder, F.Cu at (24.8, 33.2)
- added C6: C_Polarized_Small, Capacitor_SMD:C_0603_1608Metric_Pad1.08x0.95mm_HandSolder, F.Cu at (31.4, 33.2)
- added C7: C_Small, Capacitor_SMD:C_0603_1608Metric_Pad1.08x0.95mm_HandSolder, F.Cu at (33.1, 33.2)
- added C8: C_Small, Capacitor_SMD:C_0603_1608Metric_Pad1.08x0.95mm_HandSolder, F.Cu at (21.6, 28.8)
- added C9: C_Polarized_Small, Capacitor_SMD:C_0603_1608Metric_Pad1.08x0.95mm_HandSolder, F.Cu at (26.8, 24.8)
- added R22: R_Small, Resistor_SMD:R_0603_1608Metric_Pad0.98x0.95mm_HandSolder, F.Cu at (18.0, 28.8)
- added R23: R_Small, Resistor_SMD:R_0603_1608Metric_Pad0.98x0.95mm_HandSolder, F.Cu at (18.0, 27.0)
- added R24: R_Small, Resistor_SMD:R_0603_1608Metric_Pad0.98x0.95mm_HandSolder, F.Cu at (25.2, 28.8)
- added U2: TCAN332, Package_SO:SOP-8_3.9x4.9mm_P1.27mm, F.Cu at (20.8, 18.8)
- added U3: TMC2209, Package_DFN_QFN:QFN-28-1EP_5x5mm_P0.5mm_EP3.75x3.75mm_ThermalVias, F.Cu at (68.4, 82.2)
- added U4: RT8110B, Package_TO_SOT_SMD:TSOT-23-8_HandSoldering, F.Cu at (20.8, 31.8)
- J1, J2, J3, J4, J5, J6, J7, J8, J9, kibuzzard-65BAB672, kibuzzard-65BAB9B6, kibuzzard-65BABB0F, kibuzzard-65BAC02F, kibuzzard-65BAC03F, kibuzzard-65BAC3BD, kibuzzard-65BAC407, kibuzzard-65BAC420, kibuzzard-65BAC429: moved to B.Cu
- moved R13 15.5 mm to (131.8, 31.5)
- moved R14 15.5 mm to (131.8, 34.0)
- moved R15 15.5 mm to (136.1, 31.5)
- moved kibuzzard-65BAC407 15.5 mm to (133.0, 53.0), turned to 180 degrees
- moved J6 12.8 mm to (134.4, 42.6), turned to 180 degrees
- moved R18 10.2 mm to (55.2, 49.8), turned to 90 degrees
- moved J1 7.50 mm to (17.0, 24.5), turned to 0 degrees
- moved J9 7.20 mm to (72.2, 87.9), turned to 180 degrees
- moved C2 5.91 mm to (155.7, 42.0)
- moved D2 5.91 mm to (157.4, 37.2)
- moved R4 5.91 mm to (159.2, 42.0)
- moved R5 5.91 mm to (159.2, 40.2)
- moved R6 5.91 mm to (155.7, 40.2)
- moved C1 5.91 mm to (43.9, 85.7)
- moved D1 5.91 mm to (45.7, 80.9)
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Connections:
- J1 pad 2: unconnected-(J1-Pad2) -> /CanBus Handling/CANL
- J1 pad 3: unconnected-(J1-Pad3) -> /CanBus Handling/CANH
- J9 pad 1: unconnected-(J9-Pad1) -> Net-(J9-Pad1)
- J9 pad 2: unconnected-(J9-Pad2) -> Net-(J9-Pad2)
- J9 pad 3: unconnected-(J9-Pad3) -> Net-(J9-Pad3)
- J9 pad 4: unconnected-(J9-Pad4) -> Net-(J9-Pad4)
Routing:
- net +24V: track 0.00 -> 13.6 mm
- net GND: track 0.00 -> 4.46 mm
- net Net-(J3-Pad2): track 0.00 -> 4.03 mm
- net Net-(D2-Pad3): track 0.00 -> 3.59 mm
- net /CanBus Handling/CANL: track 0.00 -> 3.33 mm
- net /CanBus Handling/CANH: track 0.00 -> 3.33 mm
- net Net-(U4-Pad5): track 0.00 -> 2.83 mm
- net Net-(U4-Pad6): track 0.00 -> 2.38 mm
- net Net-(U4-Pad1): track 0.00 -> 2.33 mm
- net Net-(J2-Pad2): track 1.75 -> 4.03 mm
- net Net-(U4-Pad8): track 0.00 -> 1.83 mm
- net +3.3V: track 0.00 -> 1.80 mm
- net /Hotend Thermistor/MCU: track 0.00 -> 1.77 mm
