File: ToolHead/ToolHead.kicad_sch (KiCad schematic)
At the start: 1 part, among them J1 CANBUS

Commit message: Moderate update. Moving to other computer.
Connections:
- net CanBus Handling/CANL: now reaches J1.2 (Pin_2)
- net CanBus Handling/CANH: now reaches J1.3 (Pin_3)
Other:
- added sheet CanBus Handling (CanBusHandling.kicad_sch)
- sheet Voltage Regulation ports: added VOUT; removed none
